Commit message: added some more links. WIP: Support for polylists

File: res/text/kr210.urdf (robot description, URDF)
Before this commit: robot kuka_arm, 11 links, 10 joints
Links:
- removed link gripper_link
- removed link left_gripper_finger_link
- removed link right_gripper_finger_link
Joints:
- removed joint gripper_joint
- removed joint left_gripper_finger_joint
- removed joint right_gripper_finger_joint
